File: Boards/CDJ-800/CDJ-800.kicad_sch (KiCad schematic)
At the start: 6 parts, among them J1 CN701, J2 CN53, U2 TXS0108EPW, U3 PCM5102A

Commit message: Switch the level converters
Parts:
- removed U2: TXS0108EPW, Package_SO:TSSOP-20_4.4x6.5mm_P0.65mm, symbol Logic_LevelTranslator:TXS0108EPW
- added U1: TXS0104EPW, Package_SO:TSSOP-14_4.4x5mm_P0.65mm, symbol Logic_LevelTranslator:TXS0104EPW
- added U2: TXB0104PW, Package_SO:TSSOP-14_4.4x5mm_P0.65mm, symbol Logic_LevelTranslator:TXB0104PW
Connections:
- net at A1.1 (GPIO0): now also U2.4 (A3)
- net GNDD: now reaches A1.13 (GND), A1.18 (GND), A1.23 (GND), A1.28 (GND), A1.3 (GND), A1.38 (GND), A1.8 (GND), J2.10 (GNDD)
- net GNDD: now also J2.11 (GNDD), J2.12 (GNDD), J2.13 (GNDD), J2.14 (GNDD), U1.7 (GND), U2.7 (GND)
- net at A1.2 (GPIO1): now also U2.3 (A2)
- net at A1.21 (GPIO16): now also U1.2 (A1)
- net at A1.22 (GPIO17): now also U1.3 (A2)
- net at A1.36 (3V3): now also U1.1 (V_{CCA}), U1.8 (OE), U2.1 (VCCA), U2.8 (OE)
- net at A1.4 (GPIO2): now also U2.5 (A4)
- net at A1.5 (GPIO3): now also U2.2 (A1)
- net +5V: now reaches D1.2 (A), J2.17 (V+5P)
- net +5V: now also U1.14 (V_{CCB}), U2.14 (VCCB)
- net +7V: now reaches J2.1 (V+7M)
- net +7V: now also J1.7 (V-7A), J2.2 (V+7M), J2.3 (V+7M)
- net +6V: now reaches J2.15 (V+6B)
- net GNDS: now reaches J2.16 (GNDS)
- net at J2.19 (TSD1): now also U2.13 (B1)
- net at J2.21 (TSCS): now also U2.12 (B2)
- net at J2.22 (CONT1): now also U1.13 (B1)
- net at J2.23 (TSDO): now also U2.11 (B3)
- net at J2.24 (CONT2): now also U1.12 (B2)
- net at J2.25 (TSCLK): now also U2.10 (B4)
- net GNDM: now reaches J2.4 (GNDM)
- net GNDM: now also J2.5 (GNDM), J2.6 (GNDM)
- net +8V: now reaches J2.7 (V+8A)
- net +8V: now also J1.5 (V+8A)
- net +3V3: now reaches J2.8 (V+3D)
- net +3V3: now also J2.9 (V+3D)
- net GNDA: now reaches J1.2 (GNDA), J1.3 (GNDA), U3.9 (AGND)
Other:
- note added: "TODO: - clamp Control input voltage to +-5v - check mute voltage and state (probably better to control that over pico) - add i2s-SPID converter (although WM8804 is EOL) - add USB-Hub - connectors for front-usb, encoder - decoupling of various GND-Signals"
- moved on the sheet: J1
