File: Boards/CDJAY100S/CDJAY100S.kicad_sch (KiCad schematic)
At the start: 78 parts, among them CN701 52492-3620, CN705 52151-1410, J1 Rotary Encoder, U1 PT6324Q, U2 TXS0108EPW, U3 CH334R, X1 12MHz

Commit message: Updated the board to have an own power supply for the DAC, and an own ADC for the Pitch fader
Parts:
- removed C1, C4: 100 n, Capacitor_SMD:C_1206_3216Metric_Pad1.33x1.80mm_HandSolder, symbol Device:C_Small
- removed C2, C3: 10 u, Capacitor_SMD:C_1206_3216Metric_Pad1.33x1.80mm_HandSolder, symbol Device:C_Small
- removed R1, R5: 10 k, Resistor_SMD:R_1206_3216Metric_Pad1.30x1.75mm_HandSolder, symbol Device:R
- removed R2, R6: 20 k, Resistor_SMD:R_1206_3216Metric_Pad1.30x1.75mm_HandSolder, symbol Device:R
- removed R3, R4: 5.1 k, Resistor_SMD:R_1206_3216Metric_Pad1.30x1.75mm_HandSolder, symbol Device:R
- removed R32, R33: 10k, Resistor_SMD:R_1206_3216Metric_Pad1.30x1.75mm_HandSolder, symbol Device:R
- added C18: 1200 p, Capacitor_SMD:C_1206_3216Metric_Pad1.33x1.80mm_HandSolder, symbol Device:C_Small
- added C20, C25, C27, C28, C34: 100 n, Capacitor_SMD:C_1206_3216Metric_Pad1.33x1.80mm_HandSolder, symbol Device:C_Small
- added C26, C29, C30, C31, C32, C33: 10 u, Capacitor_SMD:C_1206_3216Metric_Pad1.33x1.80mm_HandSolder, symbol Device:C_Small
- added R17, R18, R19: 5.1k, Resistor_SMD:R_1206_3216Metric_Pad1.30x1.75mm_HandSolder, symbol Device:R_Small
- added U4: AP2127K-3.3, Package_TO_SOT_SMD:SOT-23-5, symbol Regulator_Linear:AP2127K-3.3
- added U5: TXS0108EPW, Package_SO:TSSOP-20_4.4x6.5mm_P0.65mm, symbol Logic_LevelTranslator:TXS0108EPW
- added U6: ADS1115IDGS, Package_SO:TSSOP-10_3x3mm_P0.5mm, symbol Analog_ADC:ADS1115IDGS
- C16: value 1 u -> 110 n
- R10, R11, R9: value 10 k -> 10k
- R14, R34: now not fitted
- U2: value TXS0108EPW -> TXB0108PW; symbol Logic_LevelTranslator:TXS0108EPW -> Logic_LevelTranslator:TXB0108PW
- renumbered CR2 to CNT2
Connections:
- net +3V3: now also i2S_Audio1.20 (DVDD), C25.2, C28.1, C31.2, U5.10 (OE), U5.2 (VCCA); no longer C11.1, C13.1, i2S_Audio1.11 (FLT)
- net +5V: now also C27.1, C32.1, C34.2, U4.1 (VIN), U4.3 (EN), U5.19 (VCCB), U6.8 (VDD)
- net ADIN: now also CN701.2 (ADIN), U6.4 (AIN0); no longer rPi1.31 (GPIO26_ADC0)
- net GND: now also C18.2, C20.2, C25.1, C27.2, C28.2, C31.1, C34.1, R17.2, R18.2, R19.2, U5.11 (GND), U6.1 (ADDR), U6.3 (GND); no longer C16.2, i2S_Audio1.3 (CPGND), rPi1.13 (GND), rPi1.18 (GND), rPi1.23 (GND), rPi1.28 (GND), rPi1.3 (GND), rPi1.38 (GND), rPi1.8 (GND)
- net GNDA: now also C11.2, C13.2, C16.2, i2S_Audio1.3 (CPGND), C26.2, C29.2, C30.2, C32.2, C33.1, U4.2 (GND)
- net JOG1: now also C18.1
- net JOG2: now also C20.1
- net at CN701.3 (CT): now also U6.5 (AIN1)
- net at rPi1.20 (GPIO15): now also U5.4 (A3); no longer R12.1
- net at U2.1 (A1), rPi1.12 (GPIO9): now also R19.1
- net at U2.3 (A2), rPi1.11 (GPIO8): now also R18.1
- net at U2.4 (A3), rPi1.10 (GPIO7): now also R17.1
- net at C16.1, i2S_Audio1.18 (LDOO): now also C26.1
- net +3V3A: now reaches i2S_Audio1.8 (AVDD)
- net +3V3A: now also C11.1, C13.1, i2S_Audio1.1 (CPVDD), i2S_Audio1.11 (FLT), C29.1, C30.1, C33.2, U4.5 (VOUT); no longer C13.2
- net at rPi1.29 (GPIO22): now also U5.3 (A2); no longer R13.1
- net CT: no longer names the net of rPi1.32 (GPIO27_ADC1)
- net CT: now also U5.9 (A8)
- new net: U5.12 (B8), U6.10 (SCL)
- new net: U5.13 (B7), U6.9 (SDA)
- new net: U5.8 (A7), rPi1.31 (GPIO26_ADC0)
- new net: rPi1.13 (GND), rPi1.18 (GND), rPi1.23 (GND), rPi1.28 (GND), rPi1.3 (GND), rPi1.38 (GND), rPi1.8 (GND)
- new net CNT1: R13.1, U5.17 (B3)
- new net CNT2: R12.1, U5.18 (B2)
Other:
- moved on the sheet: C11, C12, C13, C16, C17, D10, D11, D12, D8, D9, J1, JP1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

Commit message: Renamed the components to consistent placement
Parts:
- removed R17, R18, R19: 5.1k, Resistor_SMD:R_1206_3216Metric_Pad1.30x1.75mm_HandSolder, symbol Device:R_Small
- renumbered C12 to C1, C22 to C10, C24 to C11, C15 to C12, C14 to C13, C23 to C14, C30 to C15, C13 to C16, C11 to C17, C29 to C18, C16 to C19, C17 to C2, C32 to C20, C33 to C21, C26 to C22, C8 to C23, C18 to C24, C7 to C25, C20 to C26, C9 to C27, C6 to C28, C5 to C29, C27 to C3, C28 to C4, C34 to C5, C19 to C6, C21 to C7, C31 to C8, C25 to C9, CN701 to CN1, CN705 to CN2, CNT2 to CNT1, D8 to D1, D9 to D2, D10 to D3, D11 to D4, D12 to D5, D14 to D6, D16 to D7, D15 to D8, D13 to D9, R7 to R1, R35 to R10, R16 to R11, R24 to R12, R25 to R13, R26 to R14, R27 to R15, R28 to R16, R29 to R17, R30 to R18, R31 to R19, R8 to R2, R12 to R21, R13 to R22, R14 to R23, R34 to R24, R37 to R25, R36 to R26, R15 to R3, R21 to R4, R22 to R5, R9 to R6, R10 to R7, R11 to R8, R23 to R9, U2 to U1, U5 to U2, U6 to U3, U1 to U5, U3 to U6

Commit message: Version 1.6
Parts:
- removed C3, C4: 100 n, Capacitor_SMD:C_1206_3216Metric_Pad1.33x1.80mm_HandSolder, symbol Device:C_Small
- removed R12, R13, R14, R15, R16, R17, R18, R19: 22k, Resistor_SMD:R_1206_3216Metric_Pad1.30x1.75mm_HandSolder, symbol Device:R
- removed R23, R24: 10k, Resistor_SMD:R_1206_3216Metric_Pad1.30x1.75mm_HandSolder, symbol Device:R
- removed U2: TXS0108EPW, Package_SO:TSSOP-20_4.4x6.5mm_P0.65mm, symbol Logic_LevelTranslator:TXS0108EPW
- C26: value 100 n -> 1200 p
- U1: value TXB0108PW -> TXS0108; symbol Logic_LevelTranslator:TXB0108PW -> Logic_LevelTranslator:TXS0108EPW
Connections:
- net +5V: now also C2.2; no longer C2.1
- net CNT1: now also U1.16 (B4)
- net CNT2: now also U1.17 (B3)
- net GND: now also C2.1, rPi1.13 (GND), rPi1.18 (GND), rPi1.23 (GND), rPi1.28 (GND), rPi1.3 (GND), rPi1.38 (GND), rPi1.8 (GND); no longer C2.2
- net KD0: now also rPi1.12 (GPIO9); no longer U1.20 (B1)
- net SPI0 CS: now also U1.9 (A8); no longer U1.5 (A4)
- net STB: now also U1.12 (B8); no longer U1.16 (B4)
- net at U3.10 (SCL): now also U1.18 (B2)
- net at U3.9 (SDA): now also U1.20 (B1)
- net at rPi1.29 (GPIO22): now also U1.4 (A3)
- net at rPi1.20 (GPIO15): now also U1.5 (A4)
- net at rPi1.31 (GPIO26_ADC0): now also U1.1 (A1)
- net at rPi1.32 (GPIO27_ADC1): now also U1.3 (A2)
- net at CN1.7 (KD2): now also rPi1.10 (GPIO7); no longer U1.17 (B3)
- net at CN1.8 (KD1): now also rPi1.11 (GPIO8); no longer U1.18 (B2)
Other:
- moved on the sheet: C1, C2
